File: BatteryBoard.kicad_sch (KiCad schematic)
At the start: 20 parts, among them J1 Conn_01x05_Pin, J2 Conn_01x05_Pin, SW1 SW_SPST, U1 BQ25619ERTWR

Commit message: Board Outline and placement Completed
Parts:
- J1, J2: footprint (none) -> Library:5_Castellated
Connections:
- net CE_N: now also J1.5 (Pin_5)
- net GND: now also J2.1 (Pin_1); no longer J2.5 (Pin_5)
- net INT_N: now also J1.4 (Pin_4)
- net SCL: now also J1.2 (Pin_2)
- net SDA: now also J1.3 (Pin_3)
- net SW: now also J2.5 (Pin_5)
- net VBUS: now also J1.1 (Pin_1)
Changed lines of the file:
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@@
-		)
-	)
-	(label "SDA"
-		(at 57.15 85.09 0)
-		(effects
-			(font
-				(size 1.27 1.27)
-			)
-			(justify left bottom)
 		)
 	)
@@
 		)
 	)
-	(label "SCL"
-		(at 57.15 87.63 0)
-		(effects
-			(font
-				(size 1.27 1.27)
-			)
-			(justify left bottom)
-		)
-	)
 	(label "INT_N"
-		(at 57.15 90.17 0)
+		(at 49.53 90.17 0)
 		(effects
 			(font
@@
 		)
 	)
-	(label "SW"
-		(at 257.81 60.96 180)
+	(label "SCL"
+		(at 49.53 85.09 0)
 		(effects
 			(font
 				(size 1.27 1.27)
 			)
-			(justify right bottom)
+			(justify left bottom)
 		)
 	)
@@
 		)
 	)
+	(label "SW"
+		(at 264.16 71.12 180)
+		(effects
+			(font
+				(size 1.27 1.27)
+			)
+			(justify right bottom)
+		)
+	)
 	(label "CE_N"
-		(at 57.15 92.71 0)
+		(at 49.53 92.71 0)
 		(effects
 			(font
@@
 		)
 	)
+	(label "SDA"
+		(at 49.53 87.63 0)
+		(effects
+			(font
+				(size 1.27 1.27)
+			)
+			(justify left bottom)
+		)
+	)
 	(label "REGN"
 		(at 152.4 72.39 0)
@@
 	(symbol
 		(lib_id "power:GND")
-		(at 264.16 71.12 0)
+		(at 264.16 60.96 180)
 		(unit 1)
 		(exclude_from_sim no)
@@
 		(fields_autoplaced yes)
 		(property "Reference" "#PWR017"
-			(at 264.16 77.47 0)
+			(at 264.16 54.61 0)
 			(effects
 				(font
@@
 		)
 		(property "Value" "GND"
-			(at 264.16 75.2531 0)
-			(effects
-				(font
-					(size 1.27 1.27)
-				)
+			(at 266.065 59.69 0)
+			(effects
+				(font
+					(size 1.27 1.27)
+				)
+				(justify right)
 			)
 		)
 		(property "Footprint" ""
-			(at 264.16 71.12 0)
+			(at 264.16 60.96 0)
 			(effects
 				(font
@@
 		)
 		(property "Datasheet" ""
-			(at 264.16 71.12 0)
+			(at 264.16 60.96 0)
 			(effects
 				(font
@@
 		)
 		(property "Description" "Power symbol creates a global label with name \"GND\" , ground"
-			(at 264.16 71.12 0)
+			(at 264.16 60.96 0)
 			(effects
 				(font
@@
 			)
 		)
-		(property "Footprint" ""
+		(property "Footprint" "Library:5_Castellated"
 			(at 44.45 87.63 0)
 			(effects
@@
 			)
 		)
-		(property "Footprint" ""
+		(property "Footprint" "Library:5_Castellated"
 			(at 269.24 66.04 0)
 			(effects
@@
 	(symbol
 		(lib_id "power:VBUS")
-		(at 57.15 82.55 0)
+		(at 49.53 82.55 0)
 		(unit 1)
 		(exclude_from_sim no)
@@
 		(fields_autoplaced yes)
 		(property "Reference" "#PWR020"
-			(at 57.15 86.36 0)
+			(at 49.53 86.36 0)
 			(effects
 				(font
@@
 		)
 		(property "Value" "VBUS"
-			(at 57.15 78.4169 0)
+			(at 49.53 78.4169 0)
 			(effects
 				(font
@@
 		)
 		(property "Footprint" ""
-			(at 57.15 82.55 0)
+			(at 49.53 82.55 0)
 			(effects
 				(font
@@
 		)
 		(property "Datasheet" ""
-			(at 57.15 82.55 0)
+			(at 49.53 82.55 0)
 			(effects
 				(font
@@
 		)
 		(property "Description" "Power symbol creates a global label with name \"VBUS\""
-			(at 57.15 82.55 0)
-			(effects
-				(font
+			(at 49.53 82.55 0)
+			(effects
+				(font

Commit message: Minor Update for Routing
Parts:
- removed D2: LED, LED_SMD:LED_0402_1005Metric, symbol Device:LED
- removed R3: 10k, Resistor_SMD:R_0402_1005Metric, symbol Device:R
Connections:
- net PG: no longer names the net of U1.3 (PMID_GOOD)
- net STAT: no longer names the net of U1.4 (STAT)
- no-connect marks 1 -> 3
Other:
- note added: "Stat expected by accompanying PCB, querying via I2C"
- note removed: "TODO PG"
Changed lines of the file:
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@@
 	(generator_version "9.0")
 	(paper "A4")
-	(text "TODO PG"
-		(exclude_from_sim no)
-		(at 69.088 136.906 0)
-		(effects
-			(font
-				(size 1.27 1.27)
-			)
-		)
-	)
 	(text "Pulled high to 500mA"
 		(exclude_from_sim no)
 		(at 86.868 113.538 90)
+		(effects
+			(font
+				(size 1.27 1.27)
+			)
+		)
+	)
+	(text "Stat expected by accompanying PCB, \nquerying via I2C"
+		(exclude_from_sim no)
+		(at 165.1 112.014 90)
 		(effects
 			(font
@@
 		(at 106.68 69.85)
 	)
+	(no_connect
+		(at 106.68 118.11)
+	)
+	(no_connect
+		(at 152.4 107.95)
+	)
 	(wire
 		(pts
@@
 	(wire
 		(pts
-			(xy 170.18 107.95) (xy 171.45 107.95)
-		)
-		(stroke
-			(width 0)
-			(type default)
-		)
-	)
-	(wire
-		(pts
 			(xy 99.06 62.23) (xy 99.06 64.77)
 		)
@@
 	(wire
 		(pts
-			(xy 171.45 107.95) (xy 171.45 104.14)
-		)
-		(stroke
-			(width 0)
-			(type default)
-		)
-	)
-	(wire
-		(pts
 			(xy 154.94 62.23) (xy 152.4 62.23)
 		)
@@
 	(wire
 		(pts
-			(xy 152.4 107.95) (xy 162.56 107.95)
+			(xy 264.16 57.15) (xy 264.16 60.96)
 		)
 		(stroke
@@
 		)
 	)
-	(label "STAT"
-		(at 156.21 107.95 0)
-		(effects
-			(font
-				(size 1.27 1.27)
-			)
-			(justify left bottom)
-		)
-	)
 	(label "INT_N"
 		(at 49.53 90.17 0)
@@
 		)
 	)
-	(label "PG"
-		(at 69.85 140.97 180)
-		(effects
-			(font
-				(size 1.27 1.27)
-			)
-			(justify right bottom)
-		)
-	)
 	(label "SW"
 		(at 152.4 97.79 0)
@@
 		)
 	)
-	(label "VSYS"
-		(at 171.45 96.52 90)
-		(effects
-			(font
-				(size 1.27 1.27)
-			)
-			(justify left bottom)
-		)
-	)
 	(label "VBAT"
 		(at 264.16 66.04 180)
@@
 			)
 			(justify left bottom)
-		)
-	)
-	(label "PG"
-		(at 106.68 118.11 180)
-		(effects
-			(font
-				(size 1.27 1.27)
-			)
-			(justify right bottom)
 		)
 	)
@@
 	(symbol
 		(lib_id "Device:R")
-		(at 166.37 107.95 90)
-		(unit 1)
-		(exclude_from_sim no)
-		(in_bom yes)
-		(on_board yes)
-		(dnp no)
-		(property "Reference" "R3"
-			(at 166.37 105.918 90)
-			(effects
-				(font
-					(size 1.27 1.27)
-				)
-			)
-		)
-		(property "Value" "10k"
-			(at 166.37 107.95 90)
-			(effects
-				(font
-					(size 1.27 1.27)
-				)
-			)
-		)
-		(property "Footprint" "Resistor_SMD:R_0402_1005Metric"
-			(at 166.37 109.728 90)
-			(effects
-				(font
-					(size 1.27 1.27)
-				)
-				(hide yes)
-			)
-		)
-		(property "Datasheet" "~"
-			(at 166.37 107.95 0)
-			(effects
-				(font
-					(size 1.27 1.27)
-				)
-				(hide yes)
-			)
-		)
-		(property "Description" "Resistor"
-			(at 166.37 107.95 0)
-			(effects
-				(font
-					(size 1.27 1.27)
-				)
-				(hide yes)
-			)
-		)
-		(pin "2"
-		)
-		(pin "1"
-		)
-		(instances
-			(project ""
-				(path "/168724d5-94e3-4977-93b0-afa14ed6e82b"
-					(reference "R3")
-					(unit 1)
-				)
-			)
-		)
-	)
-	(symbol
-		(lib_id "Device:R")
 		(at 198.12 129.54 180)
 		(unit 1)
@@
 	(symbol
 		(lib_id "power:GND")
-		(at 264.16 60.96 180)
+		(at 264.16 57.15 180)
 		(unit 1)
 		(exclude_from_sim no)
@@
 		(fields_autoplaced yes)
 		(property "Reference" "#PWR017"
-			(at 264.16 54.61 0)
+			(at 264.16 50.8 0)
 			(effects
 				(font
@@
 		)
 		(property "Value" "GND"
-			(at 266.065 59.69 0)
+			(at 266.065 55.88 0)
 			(effects
 				(font
@@
 		)
 		(property "Footprint" ""
-			(at 264.16 60.96 0)
+			(at 264.16 57.15 0)
 			(effects
 				(font
@@
 		)
 		(property "Datasheet" ""
-			(at 264.16 60.96 0)
+			(at 264.16 57.15 0)
 			(effects
 				(font
@@
 		)
 		(property "Description" "Power symbol creates a global label with name \"GND\" , ground"
-			(at 264.16 60.96 0)
+			(at 264.16 57.15 0)
 			(effects
 				(font
@@
 					(unit 1)
 				)
-			)
-		)
-	)
-	(symbol
-		(lib_id "Device:LED")
-		(at 171.45 100.33 90)
-		(unit 1)
-		(exclude_from_sim no)
-		(in_bom yes)
-		(on_board yes)
-		(dnp no)
-		(fields_autoplaced yes)
-		(property "Reference" "D2"
-			(at 174.371 100.7053 90)
-			(effects
-				(font
-					(size 1.27 1.27)
-				)
-				(justify right)
-			)
-		)
-		(property "Value" "LED"
-			(at 174.371 103.1296 90)
-			(effects
-				(font
-					(size 1.27 1.27)
-				)
-				(justify right)
-			)
-		)
-		(property "Footprint" "LED_SMD:LED_0402_1005Metric"
-			(at 171.45 100.33 0)
-			(effects
-				(font
-					(size 1.27 1.27)
-				)
-				(hide yes)
-			)
-		)
-		(property "Datasheet" "~"
-			(at 171.45 100.33 0)
-			(effects
-				(font
-					(size 1.27 1.27)
-				)
-				(hide yes)
-			)
-		)
-		(property "Description" "Light emitting diode"
-			(at 171.45 100.33 0)
-			(effects
-				(font
-					(size 1.27 1.27)
-				)
-				(hide yes)
-			)
-		)
-		(property "Sim.Pins" "1=K 2=A"
-			(at 171.45 100.33 0)
-			(effects
-				(font
-					(size 1.27 1.27)
-				)
-				(hide yes)
-			)
-		)
-		(pin "2"
-		)
-		(pin "1"
-		)
-		(instances
-			(project ""
-				(path "/168724d5-94e3-4977-93b0-afa14ed6e82b"
-					(reference "D2")
-					(unit 1)
-				)

Commit message: Out to Review
Connections:
- net SW: now also C7.1, L1.1, U1.19 (SW), U1.20 (SW); no longer J2.5 (Pin_5), SW1.2 (B), U1.12 (QON_N)
- net BUTTON: now reaches J2.4 (Pin_4)
- net BUTTON: now also SW1.2 (B), U1.12 (QON_N); no longer R5.2
- new net TS_BAT: J2.5 (Pin_5), R5.2
Other:
- moved on the sheet: R5
Changed lines of the file:
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@@
+	(wire
+		(pts
+			(xy 251.46 71.12) (xy 264.16 71.12)
+		)
+		(stroke
+			(width 0)
+			(type default)
+		)
+	)
 	(wire
 		(pts
@@
 		(pts
 			(xy 106.68 113.03) (xy 90.17 113.03)
-		)
-		(stroke
-			(width 0)
-			(type default)
-		)
-	)
-	(wire
-		(pts
-			(xy 259.08 68.58) (xy 264.16 68.58)
 		)
 		(stroke
@@
 		)
 	)
+	(label "TS"
+		(at 243.84 71.12 180)
+		(effects
+			(font
+				(size 1.27 1.27)
+			)
+			(justify right bottom)
+		)
+	)
 	(label "VSYS"
 		(at 167.64 60.96 0)
@@
 		)
 	)
-	(label "SW"
-		(at 185.42 97.79 180)
-		(effects
-			(font
-				(size 1.27 1.27)
-			)
-			(justify right bottom)
-		)
-	)
 	(label "VBAT"
 		(at 203.2 80.01 90)
@@
 		)
 	)
+	(label "BUTTON"
+		(at 152.4 97.79 0)
+		(effects
+			(font
+				(size 1.27 1.27)
+			)
+			(justify left bottom)
+		)
+	)
 	(label "SCL"
 		(at 106.68 87.63 180)
@@
 		)
 	)
+	(label "BUTTON"
+		(at 264.16 68.58 180)
+		(effects
+			(font
+				(size 1.27 1.27)
+			)
+			(justify right bottom)
+		)
+	)
 	(label "REGN"
 		(at 173.99 120.65 90)
@@
 		)
 	)
+	(label "SW"
+		(at 154.94 59.69 90)
+		(effects
+			(font
+				(size 1.27 1.27)
+			)
+			(justify left bottom)
+		)
+	)
 	(label "PMID"
 		(at 72.39 55.88 90)
@@
 		)
 	)
-	(label "SW"
-		(at 152.4 97.79 0)
+	(label "TS_BAT"
+		(at 255.27 71.12 90)
 		(effects
 			(font
@@
 		)
 	)
-	(label "TS"
-		(at 251.46 68.58 180)
-		(effects
-			(font
-				(size 1.27 1.27)
-			)
-			(justify right bottom)
-		)
-	)
 	(label "VBAT"
 		(at 152.4 92.71 0)
@@
 		)
 	)
-	(label "SW"
-		(at 264.16 71.12 180)
-		(effects
-			(font
-				(size 1.27 1.27)
-			)
-			(justify right bottom)
-		)
-	)
 	(label "CE_N"
 		(at 49.53 92.71 0)
@@
 	(label "VBAT"
 		(at 193.04 80.01 90)
+		(effects
+			(font
+				(size 1.27 1.27)
+			)
+			(justify left bottom)
+		)
+	)
+	(label "BUTTON"
+		(at 185.42 97.79 90)
 		(effects
 			(font
@@
 	(symbol
 		(lib_id "Device:R")
-		(at 255.27 68.58 90)
+		(at 247.65 71.12 90)
 		(unit 1)
 		(exclude_from_sim no)
@@
 		(dnp yes)
 		(property "Reference" "R5"
-			(at 255.27 66.548 90)
+			(at 247.65 69.088 90)
 			(effects
 				(font
@@
 		)
 		(property "Value" "0"
-			(at 255.27 68.58 90)
+			(at 247.65 71.12 90)
 			(effects
 				(font
@@
 		)
 		(property "Footprint" "Resistor_SMD:R_0402_1005Metric"
-			(at 255.27 70.358 90)
+			(at 247.65 72.898 90)
 			(effects
 				(font
@@
 		)
 		(property "Datasheet" "~"
-			(at 255.27 68.58 0)
+			(at 247.65 71.12 0)
 			(effects
 				(font
@@
 		)
 		(property "Description" "Resistor"
-			(at 255.27 68.58 0)
-			(effects
-				(font
+			(at 247.65 71.12 0)
+			(effects
+				(font

Commit message: BOM Continuation
Parts:
- C1: Digikey Link (none) -> https://www.digikey.com/en/products/detail/samsung-electro-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; LCSC Link (none) -> https://www.lcsc.com/product-detail/C52923.html?s_z=n_CL05A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; Mfger Part# (none) -> CL05A105KA5NQNC
- C2, C3, C4, C5, C6, C8, C9: Digikey Link (none) -> https://www.digikey.com/en/products/detail/samsung-electro-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; LCSC Link (none) -> https://www.lcsc.com/product-detail/C318563.html?s_z=n_CL05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; Mfger Part# (none) -> CL05A475MO5NUNC
- R1: Digikey Link (none) -> https://www.digikey.com/en/products/detail/yageo/RC0402FR-0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; LCSC Link (none) -> https://www.lcsc.com/product-detail/C60491.html?s_z=n_RC040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; Mfger Part# (none) -> RC0402FR-07100KL
- R4: Digikey Link (none) -> https://www.digikey.com/en/products/detail/yageo/RC0402JR-0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; LCSC Link (none) -> https://www.lcsc.com/product-detail/C60489.html?s_z=n_RC040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; Mfger Part# (none) -> RC0402JR-0710KL
- SW1: Digikey Link (none) -> https://www.digikey.com/en/products/detail/c-k/NANOT-240-AS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; LCSC Link (none) -> https://www.lcsc.com/product-detail/C2760982.html?s_z=n_NAN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; Mfger Part# (none) -> NANOT 240 AS
Other:
- note removed: "Stat expected by accompanying PCB, querying via I2C"
- moved on the sheet: R1

Commit message: BOM Update
Parts:
- C7: Digikey Link (none) -> https://www.digikey.com/en/products/detail/samsung-electro-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; LCSC Link (none) -> https://www.lcsc.com/product-detail/C307339.html?s_z=n_CL05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; Mfger Part# (none) -> CL05B473KB5VPNC
- J1, J2, R5: now left out of the parts list
- L1: Digikey Link (none) -> https://www.digikey.com/en/products/detail/murata-electroni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; LCSC Link (none) -> https://www.lcsc.com/product-detail/C162587.html; Mfger Part# (none) -> LQM2HPN1R0MGHL
- R2: Digikey Link (none) -> https://www.digikey.com/en/products/detail/yageo/RC0402FR-0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; LCSC Link (none) -> https://www.lcsc.com/product-detail/C60491.html?s_z=n_RC040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; Mfger Part# (none) -> RC0402FR-07100KL; now left out of the parts list
- U1: Digikey Link (none) -> https://www.digikey.com/en/products/detail/texas-instrument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; LCSC Link (none) -> https://www.lcsc.com/product-detail/C2873446.html?s_z=n_BQ2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; Mfger Part# (none) -> BQ25619ERTWR
Changed lines of the file:
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@@
 		(unit 1)
 		(exclude_from_sim no)
-		(in_bom yes)
+		(in_bom no)
 		(on_board yes)
 		(dnp no)
@@
 			)
 		)
-		(property "Digikey Link" ""
+		(property "Digikey Link" "https://www.digikey.com/en/products/detail/samsung-electro-mechanics/CL05B473KB5VPNC/11487772"
 			(at 158.75 64.77 0)
 			(effects
@@
 			)
 		)
-		(property "LCSC Link" ""
+		(property "LCSC Link" "https://www.lcsc.com/product-detail/C307339.html?s_z=n_CL05B473KB5VPNC"
 			(at 158.75 64.77 0)
 			(effects
@@
 			)
 		)
-		(property "Mfger Part#" ""
+		(property "Mfger Part#" "CL05B473KB5VPNC"
 			(at 158.75 64.77 0)
 			(effects
@@
 		(unit 1)
 		(exclude_from_sim no)
-		(in_bom yes)
+		(in_bom no)
 		(on_board yes)
 		(dnp no)
@@
 		(unit 1)
 		(exclude_from_sim no)
-		(in_bom yes)
+		(in_bom no)
 		(on_board yes)
 		(dnp yes)
@@
 			)
 		)
-		(property "Digikey Link" ""
+		(property "Digikey Link" "https://www.digikey.com/en/products/detail/yageo/RC0402FR-07100KL/726526"
 			(at 90.17 118.11 0)
 			(effects
@@
 			)
 		)
-		(property "LCSC Link" ""
+		(property "LCSC Link" "https://www.lcsc.com/product-detail/C60491.html?s_z=n_RC0402FR-07100KL"
 			(at 90.17 118.11 0)
 			(effects
@@
 			)
 		)
-		(property "Mfger Part#" ""
+		(property "Mfger Part#" "RC0402FR-07100KL"
 			(at 90.17 118.11 0)
 			(effects
@@
 			)
 		)
-		(property "Digikey Link" ""
+		(property "Digikey Link" "https://www.digikey.com/en/products/detail/texas-instruments/BQ25619ERTWR/13545367?s=N4IgTCBcDaIEIEUwFYBsBGAnAUQEoBUB1XEAXQF8g"
 			(at 129.54 92.71 0)
 			(effects
@@
 			)
 		)
-		(property "LCSC Link" ""
+		(property "LCSC Link" "https://www.lcsc.com/product-detail/C2873446.html?s_z=n_BQ25619ERTWR"
 			(at 129.54 92.71 0)
 			(effects
@@
 			)
 		)
-		(property "Mfger Part#" ""
+		(property "Mfger Part#" "BQ25619ERTWR"
 			(at 129.54 92.71 0)
 			(effects
@@
 		(unit 1)
 		(exclude_from_sim no)
-		(in_bom yes)
+		(in_bom no)
 		(on_board yes)
 		(dnp yes)
@@
 			)
 		)
-		(property "Description" "74479787210A"
+		(property "Description" "LQM2HPN1R0MGHL"
 			(at 163.83 60.96 0)
 			(effects
@@
 			)
 		)
-		(property "Digikey Link" ""
+		(property "Digikey Link" "https://www.digikey.com/en/products/detail/murata-electronics/LQM2HPN1R0MGHL/4905781?s=N4IgTCBcDaIDIEUCyYASAFAcgRgEoAYkBxVOEAXQF8g#product-details-substitutes"
 			(at 163.83 60.96 90)
 			(effects
@@
 			)
 		)
-		(property "LCSC Link" ""
+		(property "LCSC Link" "https://www.lcsc.com/product-detail/C162587.html"
 			(at 163.83 60.96 90)
 			(effects
@@
 			)
 		)
-		(property "Mfger Part#" ""
+		(property "Mfger Part#" "LQM2HPN1R0MGHL"
 			(at 163.83 60.96 90)
 			(effects
