File: BatteryBoard.kicad_sch (KiCad schematic)
At the start: 18 parts, among them J1 Conn_01x05_Pin, J2 Conn_01x05_Pin, SW1 SW_SPST, U1 BQ25619ERTWR

Commit message: Missed Pull up for TS, updated Bulk caps to 10u, and added more DNP
Parts:
- added R3: 10k, Resistor_SMD:R_0402_1005Metric, symbol Device:R
- C2, C4, C6, C8: value 4.7u -> 10u; Digikey Link https://www.digikey.com/en/products/detail/samsung-electro-mechanics/CL05A475MO5NUNC/5961320?s=N4IgTCBcDaIMIBkAMBWAggFgOwoLIHkUA5AVSLhAF0BfIA -> https://www.digikey.com/en/products/detail/samsung-electro-mechanics/CL05A106MP8NUB8/5961314; LCSC Link https://www.lcsc.com/product-detail/C318563.html?s_z=n_CL05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 -> https://www.lcsc.com/product-detail/C307415.html?s_z=n_CL05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; Mfger Part# CL05A475MO5NUNC -> CL05A106MP8NUB8
- C3, C5, C9: value 4.7u -> 10u; Digikey Link https://www.digikey.com/en/products/detail/samsung-electro-mechanics/CL05A475MO5NUNC/5961320?s=N4IgTCBcDaIMIBkAMBWAggFgOwoLIHkUA5AVSLhAF0BfIA -> https://www.digikey.com/en/products/detail/samsung-electro-mechanics/CL05A106MP8NUB8/5961314; LCSC Link https://www.lcsc.com/product-detail/C318563.html?s_z=n_CL05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 -> https://www.lcsc.com/product-detail/C307415.html?s_z=n_CL05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; Mfger Part# CL05A475MO5NUNC -> CL05A106MP8NUB8; now not fitted
Connections:
- net REGN: now also R3.2
- net TS: now also R3.1
Changed lines of the file:
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@@
 		)
 	)
+	(label "REGN"
+		(at 171.45 97.79 90)
+		(effects
+			(font
+				(size 1.27 1.27)
+			)
+			(justify left bottom)
+		)
+	)
 	(label "TS"
 		(at 243.84 71.12 180)
@@
 		)
 	)
+	(label "TS"
+		(at 171.45 105.41 270)
+		(effects
+			(font
+				(size 1.27 1.27)
+			)
+			(justify right bottom)
+		)
+	)
 	(label "SW"
 		(at 154.94 59.69 90)
@@
 		(in_bom yes)
 		(on_board yes)
-		(dnp no)
+		(dnp yes)
 		(fields_autoplaced yes)
 		(property "Reference" "C5"
@@
 			)
 		)
-		(property "Value" "4.7u"
+		(property "Value" "10u"
 			(at 199.771 69.7921 0)
 			(effects
@@
 			)
 		)
-		(property "Digikey Link" "https://www.digikey.com/en/products/detail/samsung-electro-mechanics/CL05A475MO5NUNC/5961320?s=N4IgTCBcDaIMIBkAMBWAggFgOwoLIHkUA5AVSLhAF0BfIA"
+		(property "Digikey Link" "https://www.digikey.com/en/products/detail/samsung-electro-mechanics/CL05A106MP8NUB8/5961314"
 			(at 196.85 68.58 0)
 			(effects
@@
 			)
 		)
-		(property "LCSC Link" "https://www.lcsc.com/product-detail/C318563.html?s_z=n_CL05A475MO5NUNC"
+		(property "LCSC Link" "https://www.lcsc.com/product-detail/C307415.html?s_z=n_CL05A106MP8NUB8"
 			(at 196.85 68.58 0)
 			(effects
@@
 			)
 		)
-		(property "Mfger Part#" "CL05A475MO5NUNC"
+		(property "Mfger Part#" "CL05A106MP8NUB8"
 			(at 196.85 68.58 0)
 			(effects
@@
 		(in_bom yes)
 		(on_board yes)
-		(dnp no)
+		(dnp yes)
 		(fields_autoplaced yes)
 		(property "Reference" "C3"
@@
 			)
 		)
-		(property "Value" "4.7u"
+		(property "Value" "10u"
 			(at 75.311 60.9021 0)
 			(effects
@@
 			)
 		)
-		(property "Digikey Link" "https://www.digikey.com/en/products/detail/samsung-electro-mechanics/CL05A475MO5NUNC/5961320?s=N4IgTCBcDaIMIBkAMBWAggFgOwoLIHkUA5AVSLhAF0BfIA"
+		(property "Digikey Link" "https://www.digikey.com/en/products/detail/samsung-electro-mechanics/CL05A106MP8NUB8/5961314"
 			(at 72.39 59.69 0)
 			(effects
@@
 			)
 		)
-		(property "LCSC Link" "https://www.lcsc.com/product-detail/C318563.html?s_z=n_CL05A475MO5NUNC"
+		(property "LCSC Link" "https://www.lcsc.com/product-detail/C307415.html?s_z=n_CL05A106MP8NUB8"
 			(at 72.39 59.69 0)
 			(effects
@@
 			)
 		)
-		(property "Mfger Part#" "CL05A475MO5NUNC"
+		(property "Mfger Part#" "CL05A106MP8NUB8"
 			(at 72.39 59.69 0)
 			(effects
@@
 			)
 		)
-		(property "Value" "4.7u"
+		(property "Value" "10u"
 			(at 65.151 60.9021 0)
 			(effects
@@
 			)
 		)
-		(property "Digikey Link" "https://www.digikey.com/en/products/detail/samsung-electro-mechanics/CL05A475MO5NUNC/5961320?s=N4IgTCBcDaIMIBkAMBWAggFgOwoLIHkUA5AVSLhAF0BfIA"
+		(property "Digikey Link" "https://www.digikey.com/en/products/detail/samsung-electro-mechanics/CL05A106MP8NUB8/5961314"
 			(at 62.23 59.69 0)
 			(effects
@@
 			)
 		)
-		(property "LCSC Link" "https://www.lcsc.com/product-detail/C318563.html?s_z=n_CL05A475MO5NUNC"
+		(property "LCSC Link" "https://www.lcsc.com/product-detail/C307415.html?s_z=n_CL05A106MP8NUB8"
 			(at 62.23 59.69 0)
 			(effects
@@
 			)
 		)
-		(property "Mfger Part#" "CL05A475MO5NUNC"
+		(property "Mfger Part#" "CL05A106MP8NUB8"
 			(at 62.23 59.69 0)
 			(effects
@@
 			)
 		)
-		(property "Value" "4.7u"
+		(property "Value" "10u"
 			(at 189.611 69.7921 0)
 			(effects
@@
 			)
 		)
-		(property "Digikey Link" "https://www.digikey.com/en/products/detail/samsung-electro-mechanics/CL05A475MO5NUNC/5961320?s=N4IgTCBcDaIMIBkAMBWAggFgOwoLIHkUA5AVSLhAF0BfIA"
+		(property "Digikey Link" "https://www.digikey.com/en/products/detail/samsung-electro-mechanics/CL05A106MP8NUB8/5961314"
 			(at 186.69 68.58 0)
 			(effects
@@
 			)
 		)
-		(property "LCSC Link" "https://www.lcsc.com/product-detail/C318563.html?s_z=n_CL05A475MO5NUNC"
+		(property "LCSC Link" "https://www.lcsc.com/product-detail/C307415.html?s_z=n_CL05A106MP8NUB8"
 			(at 186.69 68.58 0)
 			(effects
@@
 			)
 		)
-		(property "Mfger Part#" "CL05A475MO5NUNC"
+		(property "Mfger Part#" "CL05A106MP8NUB8"
 			(at 186.69 68.58 0)
 			(effects
@@
 		(in_bom yes)
 		(on_board yes)
-		(dnp no)
+		(dnp yes)
 		(fields_autoplaced yes)
 		(property "Reference" "C9"
@@
 			)
 		)
-		(property "Value" "4.7u"
+		(property "Value" "10u"
 			(at 206.121 85.0321 0)
 			(effects
@@
 			)
 		)
-		(property "Digikey Link" "https://www.digikey.com/en/products/detail/samsung-electro-mechanics/CL05A475MO5NUNC/5961320?s=N4IgTCBcDaIMIBkAMBWAggFgOwoLIHkUA5AVSLhAF0BfIA"
+		(property "Digikey Link" "https://www.digikey.com/en/products/detail/samsung-electro-mechanics/CL05A106MP8NUB8/5961314"
 			(at 203.2 83.82 0)
 			(effects
@@
 			)
 		)
-		(property "LCSC Link" "https://www.lcsc.com/product-detail/C318563.html?s_z=n_CL05A475MO5NUNC"
+		(property "LCSC Link" "https://www.lcsc.com/product-detail/C307415.html?s_z=n_CL05A106MP8NUB8"
 			(at 203.2 83.82 0)
 			(effects
@@
 			)
 		)
-		(property "Mfger Part#" "CL05A475MO5NUNC"
+		(property "Mfger Part#" "CL05A106MP8NUB8"
 			(at 203.2 83.82 0)
 			(effects
@@
 			)
 		)
-		(property "Value" "4.7u"
+		(property "Value" "10u"
 			(at 195.961 85.0321 0)
 			(effects
@@
 			)
 		)
-		(property "Digikey Link" "https://www.digikey.com/en/products/detail/samsung-electro-mechanics/CL05A475MO5NUNC/5961320?s=N4IgTCBcDaIMIBkAMBWAggFgOwoLIHkUA5AVSLhAF0BfIA"
+		(property "Digikey Link" "https://www.digikey.com/en/products/detail/samsung-electro-mechanics/CL05A106MP8NUB8/5961314"
 			(at 193.04 83.82 0)
 			(effects
@@
 			)
 		)
-		(property "LCSC Link" "https://www.lcsc.com/product-detail/C318563.html?s_z=n_CL05A475MO5NUNC"
+		(property "LCSC Link" "https://www.lcsc.com/product-detail/C307415.html?s_z=n_CL05A106MP8NUB8"
 			(at 193.04 83.82 0)
 			(effects
@@
 			)
 		)
-		(property "Mfger Part#" "CL05A475MO5NUNC"
+		(property "Mfger Part#" "CL05A106MP8NUB8"
 			(at 193.04 83.82 0)
 			(effects
@@
 	)
 	(symbol
+		(lib_id "Device:R")
+		(at 171.45 101.6 180)
+		(unit 1)
+		(exclude_from_sim no)
+		(in_bom yes)
+		(on_board yes)
+		(dnp no)
+		(property "Reference" "R3"
+			(at 169.418 101.6 90)
+			(effects
+				(font
+					(size 1.27 1.27)
+				)
+			)
+		)
+		(property "Value" "10k"
+			(at 171.45 101.6 90)
+			(effects
+				(font
+					(size 1.27 1.27)
+				)
+			)
+		)
+		(property "Footprint" "Resistor_SMD:R_0402_1005Metric"
+			(at 173.228 101.6 90)
+			(effects
+				(font
+					(size 1.27 1.27)
+				)
+				(hide yes)
+			)
+		)
+		(property "Datasheet" "~"
+			(at 171.45 101.6 0)
+			(effects
+				(font
+					(size 1.27 1.27)
+				)
+				(hide yes)
+			)
+		)
+		(property "Description" "Resistor"
+			(at 171.45 101.6 0)
+			(effects
+				(font
+					(size 1.27 1.27)
+				)
+				(hide yes)
+			)
+		)
+		(property "Digikey Link" "https://www.digikey.com/en/products/detail/yageo/RC0402JR-0710KL/726418"
+			(at 171.45 101.6 90)
+			(effects
+				(font
+					(size 1.27 1.27)
+				)
+				(hide yes)
+			)
+		)
+		(property "LCSC Link" "https://www.lcsc.com/product-detail/C60489.html?s_z=n_RC0402JR-0710KL"
+			(at 171.45 101.6 90)
+			(effects
+				(font
+					(size 1.27 1.27)
+				)
+				(hide yes)
+			)
+		)
+		(property "Mfger Part#" "RC0402JR-0710KL"
+			(at 171.45 101.6 90)
+			(effects
+				(font
+					(size 1.27 1.27)
+				)
+				(hide yes)
+			)
+		)
+		(pin "2"
+		)
+		(pin "1"
+		)
+		(instances
+			(project "BatteryBoard"
+				(path "/168724d5-94e3-4977-93b0-afa14ed6e82b"
+					(reference "R3")
+					(unit 1)
+				)
+			)
+		)
+	)
+	(symbol
 		(lib_id "Device:L")
 		(at 163.83 60.96 90)
@@
 			)
 		)
-		(property "Value" "4.7u"
+		(property "Value" "10u"
 			(at 176.911 125.6721 0)
 			(effects
@@
 			)
 		)
-		(property "Digikey Link" "https://www.digikey.com/en/products/detail/samsung-electro-mechanics/CL05A475MO5NUNC/5961320?s=N4IgTCBcDaIMIBkAMBWAggFgOwoLIHkUA5AVSLhAF0BfIA"
+		(property "Digikey Link" "https://www.digikey.com/en/products/detail/samsung-electro-mechanics/CL05A106MP8NUB8/5961314"
 			(at 173.99 124.46 0)
 			(effects
@@
 			)
 		)
-		(property "LCSC Link" "https://www.lcsc.com/product-detail/C318563.html?s_z=n_CL05A475MO5NUNC"
+		(property "LCSC Link" "https://www.lcsc.com/product-detail/C307415.html?s_z=n_CL05A106MP8NUB8"
 			(at 173.99 124.46 0)
 			(effects
@@
 			)
 		)
-		(property "Mfger Part#" "CL05A475MO5NUNC"
+		(property "Mfger Part#" "CL05A106MP8NUB8"
 			(at 173.99 124.46 0)
 			(effects

Commit message: Castelated edges upodate, relayout for TS Resistor
Parts:
- removed SW1: SW_SPST, Library:NANOT 240 AS, symbol Switch:SW_SPST
Changed lines of the file:
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@@
-		)
-	)
-	(label "BUTTON"
-		(at 185.42 97.79 90)
-		(effects
-			(font
-				(size 1.27 1.27)
-			)
-			(justify left bottom)
 		)
 	)
@@
 	)
 	(symbol
-		(lib_id "Switch:SW_SPST")
-		(at 185.42 102.87 90)
-		(unit 1)
-		(exclude_from_sim no)
-		(in_bom yes)
-		(on_board yes)
-		(dnp no)
-		(fields_autoplaced yes)
-		(property "Reference" "SW1"
-			(at 186.563 101.6578 90)
-			(effects
-				(font
-					(size 1.27 1.27)
-				)
-				(justify right)
-			)
-		)
-		(property "Value" "SW_SPST"
-			(at 186.563 104.0821 90)
-			(effects
-				(font
-					(size 1.27 1.27)
-				)
-				(justify right)
-			)
-		)
-		(property "Footprint" "Library:NANOT 240 AS"
-			(at 185.42 102.87 0)
-			(effects
-				(font
-					(size 1.27 1.27)
-				)
-				(hide yes)
-			)
-		)
-		(property "Datasheet" "~"
-			(at 185.42 102.87 0)
-			(effects
-				(font
-					(size 1.27 1.27)
-				)
-				(hide yes)
-			)
-		)
-		(property "Description" "NANOT 240 AS"
-			(at 185.42 102.87 0)
-			(effects
-				(font
-					(size 1.27 1.27)
-				)
-				(hide yes)
-			)
-		)
-		(property "Digikey Link" "https://www.digikey.com/en/products/detail/c-k/NANOT-240-AS/13182173?s=N4IgTCBcDaIHIEE4HkAqACMAWADOhAyiALoC%2BQA"
-			(at 185.42 102.87 90)
-			(effects
-				(font
-					(size 1.27 1.27)
-				)
-				(hide yes)
-			)
-		)
-		(property "LCSC Link" "https://www.lcsc.com/product-detail/C2760982.html?s_z=n_NANOT"
-			(at 185.42 102.87 90)
-			(effects
-				(font
-					(size 1.27 1.27)
-				)
-				(hide yes)
-			)
-		)
-		(property "Mfger Part#" "NANOT 240 AS"
-			(at 185.42 102.87 90)
-			(effects
-				(font
-					(size 1.27 1.27)
-				)
-				(hide yes)
-			)
-		)
-		(pin "1"
-		)
-		(pin "2"
-		)
-		(instances
-			(project ""
-				(path "/168724d5-94e3-4977-93b0-afa14ed6e82b"
-					(reference "SW1")
-					(unit 1)
-				)
-			)
-		)
-	)
-	(symbol
 		(lib_id "Connector:Conn_01x05_Pin")
 		(at 44.45 87.63 0)
@@
 					(unit 1)
 				)
-			)
-		)
-	)
-	(symbol
-		(lib_id "power:GND")
-		(at 185.42 107.95 0)
-		(unit 1)
-		(exclude_from_sim no)
-		(in_bom yes)
-		(on_board yes)
-		(dnp no)
-		(fields_autoplaced yes)
-		(property "Reference" "#PWR016"
-			(at 185.42 114.3 0)
-			(effects
-				(font
-					(size 1.27 1.27)
-				)
-				(hide yes)
-			)
-		)
-		(property "Value" "GND"
-			(at 185.42 112.0831 0)
-			(effects
-				(font
-					(size 1.27 1.27)
-				)
-			)
-		)
-		(property "Footprint" ""
-			(at 185.42 107.95 0)
-			(effects
-				(font
-					(size 1.27 1.27)
-				)
-				(hide yes)
-			)
-		)
-		(property "Datasheet" ""
-			(at 185.42 107.95 0)
-			(effects
-				(font
-					(size 1.27 1.27)
-				)
-				(hide yes)
-			)
-		)
-		(property "Description" "Power symbol creates a global label with name \"GND\" , ground"
-			(at 185.42 107.95 0)
-			(effects
-				(font
-					(size 1.27 1.27)
-				)
-				(hide yes)
-			)
-		)
-		(pin "1"
-		)
-		(instances
-			(project "BatteryBoard"
-				(path "/168724d5-94e3-4977-93b0-afa14ed6e82b"
-					(reference "#PWR016")
-					(unit 1)
-				)

Commit message: Gerbers and Output Files
Parts:
- C8: now not fitted
- C9: now fitted
Changed lines of the file:
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@@
 	)
 	(label "VBAT"
-		(at 203.2 80.01 90)
+		(at 193.04 82.55 90)
 		(effects
 			(font
@@
 	)
 	(label "VBAT"
-		(at 193.04 80.01 90)
+		(at 204.47 82.55 90)
 		(effects
 			(font
@@
 	(symbol
 		(lib_id "power:GND")
-		(at 193.04 87.63 0)
+		(at 204.47 90.17 0)
 		(unit 1)
 		(exclude_from_sim no)
@@
 		(fields_autoplaced yes)
 		(property "Reference" "#PWR012"
-			(at 193.04 93.98 0)
+			(at 204.47 96.52 0)
 			(effects
 				(font
@@
 		)
 		(property "Value" "GND"
-			(at 193.04 91.7631 0)
+			(at 204.47 94.3031 0)
 			(effects
 				(font
@@
 		)
 		(property "Footprint" ""
-			(at 193.04 87.63 0)
+			(at 204.47 90.17 0)
 			(effects
 				(font
@@
 		)
 		(property "Datasheet" ""
-			(at 193.04 87.63 0)
+			(at 204.47 90.17 0)
 			(effects
 				(font
@@
 		)
 		(property "Description" "Power symbol creates a global label with name \"GND\" , ground"
-			(at 193.04 87.63 0)
+			(at 204.47 90.17 0)
 			(effects
 				(font
@@
 	(symbol
 		(lib_id "Device:C")
-		(at 203.2 83.82 0)
+		(at 193.04 86.36 0)
 		(unit 1)
 		(exclude_from_sim no)
 		(in_bom yes)
 		(on_board yes)
-		(dnp yes)
+		(dnp no)
 		(fields_autoplaced yes)
 		(property "Reference" "C9"
-			(at 206.121 82.6078 0)
+			(at 195.961 85.1478 0)
 			(effects
 				(font
@@
 		)
 		(property "Value" "10u"
-			(at 206.121 85.0321 0)
+			(at 195.961 87.5721 0)
 			(effects
 				(font
@@
 		)
 		(property "Footprint" "Capacitor_SMD:C_0402_1005Metric"
-			(at 204.1652 87.63 0)
+			(at 194.0052 90.17 0)
 			(effects
 				(font
@@
 		)
 		(property "Datasheet" "~"
-			(at 203.2 83.82 0)
+			(at 193.04 86.36 0)
 			(effects
 				(font
@@
 		)
 		(property "Description" "CL05A475MO5NUNC"
-			(at 203.2 83.82 0)
+			(at 193.04 86.36 0)
 			(effects
 				(font
@@
 		)
 		(property "Digikey Link" "https://www.digikey.com/en/products/detail/samsung-electro-mechanics/CL05A106MP8NUB8/5961314"
-			(at 203.2 83.82 0)
+			(at 193.04 86.36 0)
 			(effects
 				(font
@@
 		)
 		(property "LCSC Link" "https://www.lcsc.com/product-detail/C307415.html?s_z=n_CL05A106MP8NUB8"
-			(at 203.2 83.82 0)
+			(at 193.04 86.36 0)
 			(effects
 				(font
@@
 		)
 		(property "Mfger Part#" "CL05A106MP8NUB8"
-			(at 203.2 83.82 0)
+			(at 193.04 86.36 0)
 			(effects
 				(font
@@
 	(symbol
 		(lib_id "Device:C")
-		(at 193.04 83.82 0)
+		(at 204.47 86.36 0)
 		(unit 1)
 		(exclude_from_sim no)
 		(in_bom yes)
 		(on_board yes)
-		(dnp no)
+		(dnp yes)
 		(fields_autoplaced yes)
 		(property "Reference" "C8"
-			(at 195.961 82.6078 0)
+			(at 207.391 85.1478 0)
 			(effects
 				(font
@@
 		)
 		(property "Value" "10u"
-			(at 195.961 85.0321 0)
+			(at 207.391 87.5721 0)
 			(effects
 				(font
@@
 		)
 		(property "Footprint" "Capacitor_SMD:C_0402_1005Metric"
-			(at 194.0052 87.63 0)
+			(at 205.4352 90.17 0)
 			(effects
 				(font
@@
 		)
 		(property "Datasheet" "~"
-			(at 193.04 83.82 0)
+			(at 204.47 86.36 0)
 			(effects
 				(font
@@
 		)
 		(property "Description" "CL05A475MO5NUNC"
-			(at 193.04 83.82 0)
+			(at 204.47 86.36 0)
 			(effects
 				(font
@@
 		)
 		(property "Digikey Link" "https://www.digikey.com/en/products/detail/samsung-electro-mechanics/CL05A106MP8NUB8/5961314"
-			(at 193.04 83.82 0)
+			(at 204.47 86.36 0)
 			(effects
 				(font
@@
 		)
 		(property "LCSC Link" "https://www.lcsc.com/product-detail/C307415.html?s_z=n_CL05A106MP8NUB8"
-			(at 193.04 83.82 0)
+			(at 204.47 86.36 0)
 			(effects
 				(font
@@
 		)
 		(property "Mfger Part#" "CL05A106MP8NUB8"
-			(at 193.04 83.82 0)
+			(at 204.47 86.36 0)
 			(effects
 				(font
@@
 	(symbol
 		(lib_id "power:GND")
-		(at 203.2 87.63 0)
+		(at 193.04 90.17 0)
 		(unit 1)
 		(exclude_from_sim no)
@@
 		(fields_autoplaced yes)
 		(property "Reference" "#PWR013"
-			(at 203.2 93.98 0)
+			(at 193.04 96.52 0)
 			(effects
 				(font
@@
 		)
 		(property "Value" "GND"
-			(at 203.2 91.7631 0)
+			(at 193.04 94.3031 0)
 			(effects
 				(font
@@
 		)
 		(property "Footprint" ""
-			(at 203.2 87.63 0)
+			(at 193.04 90.17 0)
 			(effects
 				(font
@@
 		)
 		(property "Datasheet" ""
-			(at 203.2 87.63 0)
+			(at 193.04 90.17 0)
 			(effects
 				(font
@@
 		)
 		(property "Description" "Power symbol creates a global label with name \"GND\" , ground"
-			(at 203.2 87.63 0)
-			(effects
-				(font
+			(at 193.04 90.17 0)
+			(effects
+				(font
