File: BatteryBoard.kicad_sch (KiCad schematic)
At the start: 18 parts, among them J1 Conn_01x05_Pin, J2 Conn_01x05_Pin, U1 BQ25619ERTWR

Commit message: Updating BOM for LCSC Part #s
Parts:
- C1: LCSC Link https://www.lcsc.com/product-detail/C52923.html?s_z=n_CL05A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 -> https://www.lcsc.com/product-detail/C52923.html; LCSC Part Number (none) -> C52923
- C2, C3, C4, C5, C6, C8, C9: LCSC Link https://www.lcsc.com/product-detail/C307415.html?s_z=n_CL05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 -> https://www.lcsc.com/product-detail/C307415.html; LCSC Part Number (none) -> C307415
- C7: LCSC Link https://www.lcsc.com/product-detail/C307339.html?s_z=n_CL05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 -> https://www.lcsc.com/product-detail/C307339.html; LCSC Part Number (none) -> C307339
- L1: LCSC Part Number (none) -> C162587
- R1, R2: LCSC Link https://www.lcsc.com/product-detail/C60491.html?s_z=n_RC040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 -> https://www.lcsc.com/product-detail/C60491.html; LCSC Part Number (none) -> C60491
- R3, R4: LCSC Link https://www.lcsc.com/product-detail/C60489.html?s_z=n_RC040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 -> https://www.lcsc.com/product-detail/C60489.html; LCSC Part Number (none) -> C60489
- U1: LCSC Link https://www.lcsc.com/product-detail/C2873446.html?s_z=n_BQ2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 -> https://www.lcsc.com/product-detail/C2873446.html; LCSC Part Number (none) -> C2873446
Changed lines of the file:
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@@
 			)
 		)
-		(property "LCSC Link" "https://www.lcsc.com/product-detail/C52923.html?s_z=n_CL05A105KA5NQNC"
+		(property "LCSC Link" "https://www.lcsc.com/product-detail/C52923.html"
 			(at 86.36 59.69 0)
 			(effects
@@
 		)
 		(property "Mfger Part#" "CL05A105KA5NQNC"
+			(at 86.36 59.69 0)
+			(effects
+				(font
+					(size 1.27 1.27)
+				)
+				(hide yes)
+			)
+		)
+		(property "LCSC Part Number" "C52923"
 			(at 86.36 59.69 0)
 			(effects
@@
 			)
 		)
-		(property "LCSC Link" "https://www.lcsc.com/product-detail/C307415.html?s_z=n_CL05A106MP8NUB8"
+		(property "LCSC Link" "https://www.lcsc.com/product-detail/C307415.html"
 			(at 196.85 68.58 0)
 			(effects
@@
 		)
 		(property "Mfger Part#" "CL05A106MP8NUB8"
+			(at 196.85 68.58 0)
+			(effects
+				(font
+					(size 1.27 1.27)
+				)
+				(hide yes)
+			)
+		)
+		(property "LCSC Part Number" "C307415"
 			(at 196.85 68.58 0)
 			(effects
@@
 			)
 		)
-		(property "LCSC Link" "https://www.lcsc.com/product-detail/C60489.html?s_z=n_RC0402JR-0710KL"
+		(property "LCSC Link" "https://www.lcsc.com/product-detail/C60489.html"
 			(at 198.12 129.54 90)
 			(effects
@@
 		)
 		(property "Mfger Part#" "RC0402JR-0710KL"
+			(at 198.12 129.54 90)
+			(effects
+				(font
+					(size 1.27 1.27)
+				)
+				(hide yes)
+			)
+		)
+		(property "LCSC Part Number" "C60489"
 			(at 198.12 129.54 90)
 			(effects
@@
 			)
 		)
-		(property "LCSC Link" "https://www.lcsc.com/product-detail/C60491.html?s_z=n_RC0402FR-07100KL"
+		(property "LCSC Link" "https://www.lcsc.com/product-detail/C60491.html"
 			(at 90.17 107.95 0)
 			(effects
@@
 		)
 		(property "Mfger Part#" "RC0402FR-07100KL"
+			(at 90.17 107.95 0)
+			(effects
+				(font
+					(size 1.27 1.27)
+				)
+				(hide yes)
+			)
+		)
+		(property "LCSC Part Number" "C60491"
 			(at 90.17 107.95 0)
 			(effects
@@
 		)
 		(property "Mfger Part#" ""
+			(at 44.45 87.63 0)
+			(effects
+				(font
+					(size 1.27 1.27)
+				)
+				(hide yes)
+			)
+		)
+		(property "LCSC Part Number" ""
 			(at 44.45 87.63 0)
 			(effects
@@
 			)
 		)
-		(property "LCSC Link" "https://www.lcsc.com/product-detail/C307339.html?s_z=n_CL05B473KB5VPNC"
+		(property "LCSC Link" "https://www.lcsc.com/product-detail/C307339.html"
 			(at 158.75 64.77 0)
 			(effects
@@
 		)
 		(property "Mfger Part#" "CL05B473KB5VPNC"
+			(at 158.75 64.77 0)
+			(effects
+				(font
+					(size 1.27 1.27)
+				)
+				(hide yes)
+			)
+		)
+		(property "LCSC Part Number" "C307339"
 			(at 158.75 64.77 0)
 			(effects
@@
 			)
 		)
-		(property "LCSC Link" "https://www.lcsc.com/product-detail/C307415.html?s_z=n_CL05A106MP8NUB8"
+		(property "LCSC Link" "https://www.lcsc.com/product-detail/C307415.html"
 			(at 72.39 59.69 0)
 			(effects
@@
 		)
 		(property "Mfger Part#" "CL05A106MP8NUB8"
+			(at 72.39 59.69 0)
+			(effects
+				(font
+					(size 1.27 1.27)
+				)
+				(hide yes)
+			)
+		)
+		(property "LCSC Part Number" "C307415"
 			(at 72.39 59.69 0)
 			(effects
@@
 		)
 		(property "Mfger Part#" ""
+			(at 269.24 66.04 0)
+			(effects
+				(font
+					(size 1.27 1.27)
+				)
+				(hide yes)
+			)
+		)
+		(property "LCSC Part Number" ""
 			(at 269.24 66.04 0)
 			(effects
@@
 			)
 		)
-		(property "LCSC Link" "https://www.lcsc.com/product-detail/C307415.html?s_z=n_CL05A106MP8NUB8"
+		(property "LCSC Link" "https://www.lcsc.com/product-detail/C307415.html"
 			(at 62.23 59.69 0)
 			(effects
@@
 		)
 		(property "Mfger Part#" "CL05A106MP8NUB8"
+			(at 62.23 59.69 0)
+			(effects
+				(font
+					(size 1.27 1.27)
+				)
+				(hide yes)
+			)
+		)
+		(property "LCSC Part Number" "C307415"
 			(at 62.23 59.69 0)
 			(effects
@@
 			)
 		)
-		(property "LCSC Link" "https://www.lcsc.com/product-detail/C60491.html?s_z=n_RC0402FR-07100KL"
+		(property "LCSC Link" "https://www.lcsc.com/product-detail/C60491.html"
 			(at 90.17 118.11 0)
 			(effects
@@
 		)
 		(property "Mfger Part#" "RC0402FR-07100KL"
+			(at 90.17 118.11 0)
+			(effects
+				(font
+					(size 1.27 1.27)
+				)
+				(hide yes)
+			)
+		)
+		(property "LCSC Part Number" "C60491"
 			(at 90.17 118.11 0)
 			(effects
@@
 			)
 		)
-		(property "LCSC Link" "https://www.lcsc.com/product-detail/C307415.html?s_z=n_CL05A106MP8NUB8"
+		(property "LCSC Link" "https://www.lcsc.com/product-detail/C307415.html"
 			(at 186.69 68.58 0)
 			(effects
@@
 		)
 		(property "Mfger Part#" "CL05A106MP8NUB8"
+			(at 186.69 68.58 0)
+			(effects
+				(font
+					(size 1.27 1.27)
+				)
+				(hide yes)
+			)
+		)
+		(property "LCSC Part Number" "C307415"
 			(at 186.69 68.58 0)
 			(effects
@@
 			)
 		)
-		(property "LCSC Link" "https://www.lcsc.com/product-detail/C307415.html?s_z=n_CL05A106MP8NUB8"
+		(property "LCSC Link" "https://www.lcsc.com/product-detail/C307415.html"
 			(at 193.04 86.36 0)
 			(effects
@@
 		)
 		(property "Mfger Part#" "CL05A106MP8NUB8"
+			(at 193.04 86.36 0)
+			(effects
+				(font
+					(size 1.27 1.27)
+				)
+				(hide yes)
+			)
+		)
+		(property "LCSC Part Number" "C307415"
 			(at 193.04 86.36 0)
 			(effects
@@
 			)
 		)
-		(property "LCSC Link" "https://www.lcsc.com/product-detail/C2873446.html?s_z=n_BQ25619ERTWR"
+		(property "LCSC Link" "https://www.lcsc.com/product-detail/C2873446.html"
 			(at 129.54 92.71 0)
 			(effects
@@
 		)
 		(property "Mfger Part#" "BQ25619ERTWR"
+			(at 129.54 92.71 0)
+			(effects
+				(font
+					(size 1.27 1.27)
+				)
+				(hide yes)
+			)
+		)
+		(property "LCSC Part Number" "C2873446"
 			(at 129.54 92.71 0)
 			(effects
@@
 			)
 		)
-		(property "LCSC Link" "https://www.lcsc.com/product-detail/C307415.html?s_z=n_CL05A106MP8NUB8"
+		(property "LCSC Link" "https://www.lcsc.com/product-detail/C307415.html"
 			(at 204.47 86.36 0)
 			(effects
@@
 		)
 		(property "Mfger Part#" "CL05A106MP8NUB8"
+			(at 204.47 86.36 0)
+			(effects
+				(font
+					(size 1.27 1.27)
+				)
+				(hide yes)
+			)
+		)
+		(property "LCSC Part Number" "C307415"
 			(at 204.47 86.36 0)
 			(effects
@@
 		)
 		(property "Mfger Part#" ""
+			(at 247.65 71.12 90)
+			(effects
+				(font
+					(size 1.27 1.27)
+				)
+				(hide yes)
+			)
+		)
+		(property "LCSC Part Number" ""
 			(at 247.65 71.12 90)
 			(effects
@@
 			)
 		)
-		(property "LCSC Link" "https://www.lcsc.com/product-detail/C60489.html?s_z=n_RC0402JR-0710KL"
+		(property "LCSC Link" "https://www.lcsc.com/product-detail/C60489.html"
 			(at 171.45 101.6 90)
 			(effects
@@
 		)
 		(property "Mfger Part#" "RC0402JR-0710KL"
+			(at 171.45 101.6 90)
+			(effects
+				(font
+					(size 1.27 1.27)
+				)
+				(hide yes)
+			)
+		)
+		(property "LCSC Part Number" "C60489"
 			(at 171.45 101.6 90)
 			(effects
@@
 			)
 		)
+		(property "LCSC Part Number" "C162587"
+			(at 163.83 60.96 90)
+			(effects
+				(font
+					(size 1.27 1.27)
+				)
+				(hide yes)
+			)
+		)
 		(pin "2"
 		)
@@
 			)
 		)
-		(property "LCSC Link" "https://www.lcsc.com/product-detail/C307415.html?s_z=n_CL05A106MP8NUB8"
+		(property "LCSC Link" "https://www.lcsc.com/product-detail/C307415.html"
 			(at 173.99 124.46 0)
 			(effects
@@
 			(at 173.99 124.46 0)
 			(effects
+				(font
+					(size 1.27 1.27)
+				)
+				(hide yes)
+			)
+		)
+		(property "LCSC Part Number" "C307415"
+			(at 173.99 124.46 0)
+			(effects

Commit message: Cleanup, and ordered boards
Parts:
- C1: LCSC Link https://www.lcsc.com/product-detail/C52923.html -> (none); LCSC Part Number C52923 -> (none); MPN (none) -> CL05A105KA5NQNC; Mfger Part# CL05A105KA5NQNC -> (none)
- C2, C3, C4, C5, C6, C8, C9: LCSC Link https://www.lcsc.com/product-detail/C307415.html -> (none); LCSC Part Number C307415 -> (none); MPN (none) -> CL05A106MP8NUB8; Mfger Part# CL05A106MP8NUB8 -> (none)
- C7: LCSC Link https://www.lcsc.com/product-detail/C307339.html -> (none); LCSC Part Number C307339 -> (none); MPN (none) -> CL05B473KB5VPNC; Mfger Part# CL05B473KB5VPNC -> (none)
- L1: value 1u -> 1uH; LCSC Link https://www.lcsc.com/product-detail/C162587.html -> (none); LCSC Part Number C162587 -> (none); MPN (none) -> LQM2HPN1R0MGHL; Mfger Part# LQM2HPN1R0MGHL -> (none)
- R1, R2: LCSC Link https://www.lcsc.com/product-detail/C60491.html -> (none); LCSC Part Number C60491 -> (none); MPN (none) -> RC0402FR-07100KL; Mfger Part# RC0402FR-07100KL -> (none)
- R3, R4: LCSC Link https://www.lcsc.com/product-detail/C60489.html -> (none); LCSC Part Number C60489 -> (none); MPN (none) -> RC0402JR-0710KL; Mfger Part# RC0402JR-0710KL -> (none)
- U1: LCSC Link https://www.lcsc.com/product-detail/C2873446.html -> (none); LCSC Part Number C2873446 -> (none); MPN (none) -> BQ25619ERTWR; Mfger Part# BQ25619ERTWR -> (none)
